File: KiCAD/RCMhardwareNibble.kicad_pcb (KiCad board)
At the start: 4 copper layers, 27.4 x 28.4 mm, 50 parts, among them IC1 TMC7300, IC2 TMC7300, J1 pads to solder wires to, J2 Conn_01x03, J3 Conn_01x03, J4 Conn_01x03, J5 Conn_01x03, J6 2x04 female header pins, J9 Conn_02x02_Top_Bottom, Q3 BSS138, N channel mosfet >=0.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

Commit message: v1.4.0
Parts:
- U1: footprint !RCMhardware footprints:pololu4085 -> !RCMhardware footprints:pololu 4085
- moved U1 2.29 mm to (140.1, 34.4)
Connections:
- U1 pad 1: vbat -> servopower
- U1 pad 3: servopower -> vbat
Other:
- board text added: "1 2 3 4"
- board text added: "v1.4"
- board text removed: "v1.3"
Changed lines of the file:
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@@
     (grid_origin 138.557 36.857)
     (pcbplotparams
-      (layerselection 0x0000030_7ffffff8)
+      (layerselection 0x000f0ff_ffffffff)
       (plot_on_all_layers_selection 0x0000000_00000000)
       (disableapertmacros false)
@@
       (sketchpadsonfab false)
       (subtractmaskfromsilk false)
-      (outputformat 3)
+      (outputformat 1)
       (mirror false)
       (drillshape 0)
       (scaleselection 1)
-      (outputdirectory "pcbway1.3/gerbers")
+      (outputdirectory "production 1.4/gerbers")
     )
   )
@@
     )
   )
-  (footprint "!RCMhardware footprints:pololu4085" (layer "F.Cu")
-    (at 141.351 36.349 -90)
+  (footprint "!RCMhardware footprints:pololu 4085" (layer "F.Cu")
+    (at 140.081 34.444 -90)
     (property "Manufacturer" "Pololu")
     (property "Package" "tht")
@@
     (property "mpn" "do not place or purchase for PCB assembly")
     (attr through_hole)
-    (fp_text reference "U1" (at -1.91 -11.33 -90 unlocked) (layer "F.SilkS") hide
+    (fp_text reference "U1" (at 4.318 -8.636 -90 unlocked) (layer "F.SilkS") hide
         (effects (font (size 1 1) (thickness 0.1)))
     )
-    (fp_text value "pololu 4085" (at 2.6924 -2.6416 -90 unlocked) (layer "F.SilkS")
-        (effects (font (size 0.8 0.8) (thickness 0.15)))
+    (fp_text value "pololu 4085" (at 0 1 -90 unlocked) (layer "F.Fab")
+        (effects (font (size 1 1) (thickness 0.15)))
+    )
+    (fp_text user "vin" (at 7.366 -2.286 unlocked) (layer "F.SilkS")
+        (effects (font (size 1 1) (thickness 0.1)) (justify left bottom))
     )
-    (fp_text user "out" (at -1.9304 -1.016 -90 unlocked) (layer "F.SilkS")
-        (effects (font (size 1 1) (thickness 0.15)) (justify left bottom))
+    (fp_text user "vout" (at 2.286 -2.286 unlocked) (layer "F.SilkS")
+        (effects (font (size 1 1) (thickness 0.1)) (justify left bottom))
     )
-    (fp_text user "gnd" (at 0.8128 -1.0668 -90 unlocked) (layer "F.SilkS")
-        (effects (font (size 1 1) (thickness 0.15)) (justify left bottom))
+    (fp_text user "gnd" (at 4.826 -2.54 unlocked) (layer "F.SilkS")
+        (effects (font (size 1 1) (thickness 0.1)) (justify left bottom))
     )
-    (fp_text user "in" (at 4.6228 -1.016 -90 unlocked) (layer "F.SilkS")
-        (effects (font (size 1 1) (thickness 0.15)) (justify left bottom))
+    (fp_text user "pololu 4085" (at 1.2954 -9.2964 -90 unlocked) (layer "F.SilkS")
+        (effects (font (size 0.8 0.8) (thickness 0.1)) (justify left bottom))
     )
-    (fp_text user "${REFERENCE}" (at -1.91 -8.33 -90 unlocked) (layer "F.Fab")
+    (fp_text user "${REFERENCE}" (at 0 2.5 -90 unlocked) (layer "F.Fab")
         (effects (font (size 1 1) (thickness 0.15)))
     )
-    (fp_rect (start -1.91 -10.83) (end 6.99 1.27)
+    (fp_rect (start 0 -11.938) (end 8.89 0)
       (stroke (width 0.1) (type default)) (fill none) (layer "F.SilkS"))
-    (pad "1" thru_hole circle (at 5.08 0 270) (size 1.524 1.524) (drill 0.762) (layers "*.Cu" "*.Mask")
-      (net 29 "vbat") (pinfunction "vin") (pintype "input"))
-    (pad "2" thru_hole rect (at 2.54 0 270) (size 1.524 1.524) (drill 0.762) (layers "*.Cu" "*.Mask")
+    (fp_rect (start 0 -11.938) (end 8.89 0)
+      (stroke (width 0.05) (type default)) (fill none) (layer "F.CrtYd"))
+    (pad "1" thru_hole circle (at 1.905 -1.27 270) (size 1.524 1.524) (drill 0.762) (layers "*.Cu" "*.Mask")
+      (net 30 "servopower") (pinfunction "vout") (pintype "power_out"))
+    (pad "2" thru_hole circle (at 4.445 -1.27 270) (size 1.524 1.524) (drill 0.762) (layers "*.Cu" "*.Mask")
       (net 1 "GND") (pinfunction "gnd") (pintype "input"))
-    (pad "3" thru_hole circle (at 0 0 270) (size 1.524 1.524) (drill 0.762) (layers "*.Cu" "*.Mask")
-      (net 30 "servopower") (pinfunction "vout") (pintype "input"))
-    (model "${KIPRJMOD}/!RCMhardware footprints/Untitled.stl.STP"
-      (offset (xyz -2 -1.25 0))
+    (pad "3" thru_hole circle (at 6.985 -1.27 270) (size 1.524 1.524) (drill 0.762) (layers "*.Cu" "*.Mask")
+      (net 29 "vbat") (pinfunction "vin") (pintype "power_in"))
+    (model "${KIPRJMOD}/!RCMhardware footprints/pololu 4085 5v-2a-step-up-step-down-voltage-regulator-s13v20f5.step"
+      (offset (xyz 0 0 2.5))
       (scale (xyz 1 1 1))
       (rotate (xyz 0 0 0))
@@
         (effects (font (size 0.8 0.8) (thickness 0.15)) (justify top))
     )
-    (fp_text user "usb" (at 0.7874 -7.96229 unlocked) (layer "F.SilkS")
+    (fp_text user "usb" (at 0 -7.112 unlocked) (layer "F.SilkS")
         (effects (font (size 2 2) (thickness 0.2)))
     )
@@
   (gr_line (start 135.001 56.669) (end 137.033 56.669)
     (stroke (width 0.15) (type default)) (layer "F.SilkS"))
+  (gr_arc (start 140.666523 40.674734) (mid 140.271184 38.921173) (end 140.639801 37.1618)
+    (stroke (width 0.15) (type default)) (layer "F.SilkS"))
   (gr_line (start 135.509 57.05) (end 135.001 56.669)
     (stroke (width 0.15) (type default)) (layer "F.SilkS"))
@@
   (gr_rect (start 127.889 34.317) (end 155.321 62.765)
     (stroke (width 0.1) (type default)) (fill none) (layer "Edge.Cuts"))
-  (gr_text "scl\n" (at 137.1346 51.7414) (layer "B.SilkS")
+  (gr_text "scl\n" (at 136.9314 51.589) (layer "B.SilkS")
     (effects (font (size 0.8 0.8) (thickness 0.1)) (justify left bottom mirror))
   )
@@
     (effects (font (size 0.8 0.8) (thickness 0.15)) (justify left bottom mirror))
   )
-  (gr_text "sda" (at 136.9822 55.399) (layer "B.SilkS")
+  (gr_text "sda" (at 136.9822 55.3482) (layer "B.SilkS")
     (effects (font (size 0.8 0.8) (thickness 0.1)) (justify left bottom mirror))
   )
@@
     (effects (font (size 0.8 0.9) (thickness 0.15)) (justify left bottom))
   )
-  (gr_text "v1.3" (at 134.5946 50.1666) (layer "F.SilkS")
+  (gr_text "v1.4" (at 134.5946 50.1666) (layer "F.SilkS")
     (effects (font (size 0.8 0.8) (thickness 0.15)) (justify left bottom))
   )
@@
     (effects (font (size 0.8 0.8) (thickness 0.15)) (justify left bottom))
   )
+  (gr_text "1  2  3  4" (at 136.0678 36.2982 -90) (layer "F.SilkS")
+    (effects (font (size 1 1) (thickness 0.15)) (justify left bottom))
+  )
   (gr_text "A  B  C  D\n" (at 142.875 56.415) (layer "F.SilkS")
