File: KiCAD/RCMhardwareNibble.kicad_sch (KiCad schematic)
At the start: 50 parts, among them IC1 TMC7300, IC2 TMC7300, J1 pads to solder wires to, J2 Conn_01x03, J3 Conn_01x03, J4 Conn_01x03, J5 Conn_01x03, J6 2x04 female header pins, J9 Conn_02x02_Top_Bottom, Q3 BSS138, N channel mosfet >=0.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

Commit message: v1.4.0
Parts:
- U1: footprint !RCMhardware footprints:pololu4085 -> !RCMhardware footprints:pololu 4085
Connections:
- net servopower: now also U1.1 (vout); no longer U1.3 (vout)
- net vbat: now also U1.3 (vin); no longer U1.1 (vin)
Other:
- title: RCM Byte -> RCM NIBBLE
Changed lines of the file:
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@@
   (paper "A2")
   (title_block
-    (title "RCM Byte")
+    (title "RCM NIBBLE")
     (company "Joshua Phelps")
+    (comment 1 "https://github.com/RCMgames/RCM-Hardware-Nibble")
   )
   (junction (at 427.99 311.15) (diameter 0) (color 0 0 0 0)
@@
     (stroke (width 0) (type default))
   )
+  (wire (pts (xy 358.14 86.36) (xy 358.14 85.09))
+    (stroke (width 0) (type default))
+  )
   (wire (pts (xy 387.35 69.85) (xy 387.35 110.49))
     (stroke (width 0) (type default))
@@
     (stroke (width 0) (type default))
   )
+  (wire (pts (xy 363.22 86.36) (xy 363.22 85.09))
+    (stroke (width 0) (type default))
+  )
   (wire (pts (xy 102.87 162.56) (xy 95.25 162.56))
     (stroke (width 0) (type default))
@@
     )
   )
-  (global_label "servopower" (shape input) (at 363.22 85.09 0) (fields_autoplaced)
-    (effects (font (size 1.27 1.27)) (justify left))
-    (property "Intersheetrefs" "${INTERSHEET_REFS}" (at 376.728 85.09 0)
-      (effects (font (size 1.27 1.27)) (justify left) hide)
-    )
-  )
   (global_label "GND" (shape bidirectional) (at 436.88 85.09 0) (fields_autoplaced)
     (effects (font (size 1.27 1.27)) (justify left))
@@
     )
   )
-  (global_label "vbat" (shape bidirectional) (at 358.14 85.09 180) (fields_autoplaced)
-    (effects (font (size 1.27 1.27)) (justify right))
-    (property "Intersheetrefs" "${INTERSHEET_REFS}" (at 350.0522 85.09 0)
-      (effects (font (size 1.27 1.27)) (justify right) hide)
-    )
-  )
   (global_label "1.8" (shape input) (at 288.29 160.02 0) (fields_autoplaced)
     (effects (font (size 1.27 1.27)) (justify left))
@@
     )
   )
+  (global_label "vbat" (shape bidirectional) (at 363.22 86.36 0) (fields_autoplaced)
+    (effects (font (size 1.27 1.27)) (justify left))
+    (property "Intersheetrefs" "${INTERSHEET_REFS}" (at 371.3078 86.36 0)
+      (effects (font (size 1.27 1.27)) (justify left) hide)
+    )
+  )
   (global_label "GND" (shape bidirectional) (at 346.71 209.55 0) (fields_autoplaced)
     (effects (font (size 1.27 1.27)) (justify left))
@@
     )
   )
+  (global_label "servopower" (shape input) (at 358.14 86.36 180) (fields_autoplaced)
+    (effects (font (size 1.27 1.27)) (justify right))
+    (property "Intersheetrefs" "${INTERSHEET_REFS}" (at 344.632 86.36 0)
+      (effects (font (size 1.27 1.27)) (justify right) hide)
+    )
+  )
   (global_label "1.8" (shape input) (at 383.54 138.43 0) (fields_autoplaced)
     (effects (font (size 1.27 1.27)) (justify left))
@@
       (effects (font (size 1.27 1.27)))
     )
-    (property "Footprint" "!RCMhardware footprints:pololu4085" (at 360.68 76.2 0)
+    (property "Footprint" "!RCMhardware footprints:pololu 4085" (at 360.68 76.2 0)
       (effects (font (size 1.27 1.27)) hide)
     )
