File: KICAD-RCM-Nibble-v1.5/RCMhardwareNibble.kicad_pcb (KiCad board)
At the start: 4 copper layers, 27.4 x 28.4 mm, 51 parts, among them IC1 TMC7300, IC2 TMC7300, J1 pads to solder wires to, J2 Conn_01x03, J3 Conn_01x03, J4 Conn_01x03, J5 Conn_01x03, J6 2x04 female header pins, J9 Conn_02x02_Top_Bottom, Q3 BSS138, N channel mosfet >=0.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

Commit message: close #3 close #4
Parts:
- C12: value 22uF/0603/>=16V -> 22uF/0603/>=10V
Changed lines of the file:
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@@
     (aux_axis_origin 138.557 36.857)
     (pcbplotparams
-      (layerselection 0x0000030_7ffffff8)
+      (layerselection 0x00010ff_ffffffff)
       (plot_on_all_layers_selection 0x0000000_00000000)
       (disableapertmacros false)
@@
       (sketchpadsonfab false)
       (subtractmaskfromsilk false)
-      (outputformat 3)
+      (outputformat 1)
       (mirror false)
       (drillshape 0)
       (scaleselection 1)
-      (outputdirectory "production1.5/")
+      (outputdirectory "production1.5/gerbers/")
     )
   )
@@
         (effects (font (size 1 1) (thickness 0.15)) (justify mirror))
     )
-    (fp_text value "22uF/0603/>=16V" (at 0 -1.43 90) (layer "B.Fab")
+    (fp_text value "22uF/0603/>=10V" (at 0 -1.43 90) (layer "B.Fab")
         (effects (font (size 1 1) (thickness 0.15)) (justify mirror))
     )
@@
     )
     (stroke (width 0.15) (type solid)) (fill solid) (layer "B.Mask"))
-  (gr_circle (center 0 47.6504) (end 0.401609 47.6504)
-    (stroke (width 0.15) (type solid)) (fill solid) (layer "B.Mask"))
   (gr_circle (center 147.4724 47.498) (end 147.8534 47.498)
