File: KICAD-RCM-Nibble-v1.5/RCMhardwareNibble.kicad_sch (KiCad schematic)
At the start: 51 parts, among them IC1 TMC7300, IC2 TMC7300, J1 pads to solder wires to, J2 Conn_01x03, J3 Conn_01x03, J4 Conn_01x03, J5 Conn_01x03, J6 2x04 female header pins, J9 Conn_02x02_Top_Bottom, Q3 BSS138, N channel mosfet >=0.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

Commit message: close #3 close #4
Parts:
- C12: value 22uF/0603/>=16V -> 22uF/0603/>=10V
Changed lines of the file:
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@@
       (effects (font (size 1.27 1.27)) (justify right))
     )
-    (property "Value" "22uF/0603/>=16V" (at 458.47 309.88 0)
+    (property "Value" "22uF/0603/>=10V" (at 458.47 309.88 0)
       (effects (font (size 1.27 1.27)) (justify right))
     )

Commit message: Update RCMhardwareNibble.kicad_sch
Parts:
- D1: Manufacturer any -> Good-Ark Semiconductor
Changed lines of the file:
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@@
       (effects (font (size 1.27 1.27)) hide)
     )
-    (property "Manufacturer" "any" (at 429.26 39.37 0)
+    (property "Manufacturer" "Good-Ark Semiconductor" (at 429.26 39.37 0)
       (effects (font (size 1.27 1.27)) hide)
     )
