File: KICAD-RCM-Nibble/RCMhardwareNibble.kicad_pcb (KiCad board)
At the start: 4 copper layers, 27.4 x 28.4 mm, 51 parts, among them IC1 TMC7300, IC2 TMC7300, J1 pads to solder wires to, J2 Conn_01x03, J3 Conn_01x03, J4 Conn_01x03, J5 Conn_01x03, J6 2x04 female header pins, J9 Conn_02x02_Top_Bottom, Q3 BSS138, N channel mosfet >=0.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

Commit message: v1.6
Other:
- board text added: "RCM Nibble v1.6"
- board text added: "v1.6"
- board text removed: "RCM Nibble v1.5"
- board text removed: "v1.5"
Changed lines of the file:
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@@
     (aux_axis_origin 138.557 36.857)
     (pcbplotparams
-      (layerselection 0x00010ff_ffffffff)
+      (layerselection 0x00010fc_ffffffff)
       (plot_on_all_layers_selection 0x0000000_00000000)
       (disableapertmacros false)
@@
       (usegerberattributes true)
       (usegerberadvancedattributes true)
-      (creategerberjobfile true)
+      (creategerberjobfile false)
       (dashed_line_dash_ratio 12.000000)
       (dashed_line_gap_ratio 3.000000)
@@
       (plotinvisibletext false)
       (sketchpadsonfab false)
-      (subtractmaskfromsilk false)
+      (subtractmaskfromsilk true)
       (outputformat 1)
       (mirror false)
       (drillshape 0)
       (scaleselection 1)
-      (outputdirectory "production1.5/gerbers/")
+      (outputdirectory "../gerbers/")
     )
   )
@@
   (gr_circle (center 143.637 45.747) (end 144.35542 45.747)
     (stroke (width 0.15) (type solid)) (fill solid) (layer "B.SilkS"))
+  (gr_line (start 152.146 36.322) (end 152.146 38.1)
+    (stroke (width 0.15) (type default)) (layer "B.SilkS"))
+  (gr_line (start 150.368 36.322) (end 152.146 36.322)
+    (stroke (width 0.15) (type default)) (layer "B.SilkS"))
+  (gr_line (start 152.146 38.1) (end 150.368 38.1)
+    (stroke (width 0.15) (type default)) (layer "B.SilkS"))
   (gr_line (start 135.509 56.288) (end 135.001 56.669)
     (stroke (width 0.15) (type default)) (layer "F.SilkS"))
@@
     (effects (font (size 2 2) (thickness 0.3)) (justify mirror))
   )
-  (gr_text "RCM Nibble v1.5\n" (at 150.6982 49.0982) (layer "B.SilkS")
+  (gr_text "RCM Nibble v1.6\n" (at 150.6982 49.0474) (layer "B.SilkS")
     (effects (font (size 0.8 0.8) (thickness 0.15)) (justify left bottom mirror))
   )
@@
     (effects (font (size 2 2) (thickness 0.3)) (justify mirror))
   )
-  (gr_text "3V\n" (at 130.6576 53.113) (layer "B.SilkS")
-    (effects (font (size 1 1) (thickness 0.15)) (justify left bottom mirror))
+  (gr_text "3V\n" (at 130.4798 52.9082) (layer "B.SilkS")
+    (effects (font (size 0.8 0.8) (thickness 0.15)) (justify left bottom mirror))
   )
   (gr_text "scl\n" (at 136.9314 51.589) (layer "B.SilkS")
     (effects (font (size 0.8 0.8) (thickness 0.1)) (justify left bottom mirror))
   )
-  (gr_text "Gnd\n" (at 130.8608 47.2964) (layer "B.SilkS")
-    (effects (font (size 0.9 0.9) (thickness 0.15)) (justify left bottom mirror))
+  (gr_text "Gnd\n" (at 130.8608 47.1424) (layer "B.SilkS")
+    (effects (font (size 0.8 0.8) (thickness 0.15)) (justify left bottom mirror))
   )
   (gr_text "TX SCL SDA A3  A2  A1  A0\n" (at 137.6934 44.5786 270) (layer "B.SilkS")
@@
     (effects (font (size 0.9 0.9) (thickness 0.15)) (justify left bottom))
   )
-  (gr_text "v1.5\n" (at 134.5946 50.1666) (layer "F.SilkS")
+  (gr_text "v1.6\n" (at 134.5946 50.1666) (layer "F.SilkS")
     (effects (font (size 0.8 0.8) (thickness 0.15)) (justify left bottom))
   )
@@
     (effects (font (size 0.8 0.8) (thickness 0.15)) (justify left bottom))
   )
-  (gr_text "3V" (at 128.8034 53.2384) (layer "F.SilkS")
+  (gr_text "3V" (at 128.8288 53.213) (layer "F.SilkS")
     (effects (font (size 0.8 0.8) (thickness 0.15)) (justify left bottom))
   )
@@
       )
     )
+  )
+  (zone (net 1) (net_name "GND") (layer "B.Cu") (hatch edge 0.5)
+    (priority 8)
+    (connect_pads yes (clearance 0))
+    (min_thickness 0.25) (filled_areas_thickness no)
+    (fill yes (thermal_gap 0.5) (thermal_bridge_width 0.5))
+    (polygon
+      (pts
+        (xy 144.8054 38.2778)
+        (xy 147.066 38.2778)
+        (xy 147.066 41.8592)
+        (xy 144.8054 41.8592)
+      )
+    )

Commit message: v1.6.1
Routing:
- net vbat: track 13.5 -> 14.1 mm
- net Net-(IC2-OA2): track 9.01 -> 8.74 mm, vias 1 -> 0
Changed lines of the file:
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@@
       (drillshape 0)
       (scaleselection 1)
-      (outputdirectory "../gerbers/")
+      (outputdirectory "../PCBproduction/gerbers/")
     )
   )
@@
     (effects (font (size 0.9 0.9) (thickness 0.15)) (justify left bottom))
   )
-  (gr_text "nibble\n" (at 133.477 49.049) (layer "F.SilkS")
+  (gr_text "nibble\n" (at 133.5024 49.049) (layer "F.SilkS")
     (effects (font (size 0.8 0.8) (thickness 0.15)) (justify left bottom))
   )
@@
     (effects (font (size 1.2 1.2) (thickness 0.15)) (justify left bottom))
   )
-  (gr_text "G  5  S\n\n" (at 129.0574 37.2888) (layer "F.SilkS")
+  (gr_text "G  5  S\n\n" (at 129.0574 37.1856) (layer "F.SilkS")
     (effects (font (size 1 1) (thickness 0.15)) (justify left bottom))
   )
@@
   (segment (start 144.916896 50.165) (end 144.29878 50.165) (width 0.25) (layer "F.Cu") (net 20))
   (segment (start 144.29878 50.165) (end 144.075 50.38878) (width 0.25) (layer "F.Cu") (net 20))
-  (segment (start 150.00538 50.168974) (end 149.79 50.384354) (width 0.25) (layer "F.Cu") (net 20))
-  (segment (start 150.111626 50.168974) (end 150.00538 50.168974) (width 0.25) (layer "F.Cu") (net 20))
+  (segment (start 149.79 50.384354) (end 149.79 50.868974) (width 0.25) (layer "F.Cu") (net 20))
+  (segment (start 150.7998 49.4808) (end 150.111626 50.168974) (width 0.25) (layer "F.Cu") (net 20))
   (segment (start 153.7228 44.5512) (end 153.797 44.477) (width 0.25) (layer "F.Cu") (net 20))
   (segment (start 150.7998 48.515973) (end 153.797 45.518773) (width 0.25) (layer "F.Cu") (net 20))
+  (segment (start 150.00538 50.168974) (end 149.79 50.384354) (width 0.25) (layer "F.Cu") (net 20))
+  (segment (start 150.111626 50.168974) (end 150.00538 50.168974) (width 0.25) (layer "F.Cu") (net 20))
   (segment (start 144.942296 50.1904) (end 144.916896 50.165) (width 0.25) (layer "F.Cu") (net 20))
-  (segment (start 150.7998 48.9204) (end 150.7998 48.515973) (width 0.25) (layer "F.Cu") (net 20))
+  (segment (start 150.7998 48.6156) (end 150.7998 49.4808) (width 0.25) (layer "F.Cu") (net 20))
   (segment (start 153.797 45.518773) (end 153.797 44.477) (width 0.25) (layer "F.Cu") (net 20))
-  (segment (start 150.7998 49.4808) (end 150.111626 50.168974) (width 0.25) (layer "F.Cu") (net 20))
   (segment (start 144.075 50.38878) (end 144.075 50.8734) (width 0.25) (layer "F.Cu") (net 20))
-  (segment (start 150.7998 48.9204) (end 150.7998 49.4808) (width 0.25) (layer "F.Cu") (net 20))
-  (segment (start 149.79 50.384354) (end 149.79 50.868974) (width 0.25) (layer "F.Cu") (net 20))
-  (via (at 150.7998 48.9204) (size 0.6) (drill 0.3) (layers "F.Cu" "B.Cu") (remove_unused_layers) (keep_end_layers) (free) (zone_layer_connections) (net 20))
+  (segment (start 150.7998 48.6156) (end 150.7998 48.515973) (width 0.25) (layer "F.Cu") (net 20))
+  (via (at 150.7998 48.6156) (size 0.6) (drill 0.3) (layers "F.Cu" "B.Cu") (remove_unused_layers) (keep_end_layers) (free) (zone_layer_connections) (net 20))
   (via (at 144.907 50.165) (size 0.6) (drill 0.3) (layers "F.Cu" "B.Cu") (remove_unused_layers) (keep_end_layers) (free) (zone_layer_connections) (net 20))
-  (segment (start 153.797 44.477) (end 151.7436 44.477) (width 0.25) (layer "B.Cu") (net 20))
-  (segment (start 151.7436 44.477) (end 151.511 44.2444) (width 0.25) (layer "B.Cu") (net 20))
-  (segment (start 150.7998 48.9204) (end 150.421189 48.541789) (width 0.25) (layer "B.Cu") (net 20))
-  (segment (start 150.421189 48.541789) (end 145.996811 48.541789) (width 0.25) (layer "B.Cu") (net 20))
   (segment (start 144.942296 49.596304) (end 144.942296 50.1904) (width 0.25) (layer "B.Cu") (net 20))
   (segment (start 145.996811 48.541789) (end 144.942296 49.596304) (width 0.25) (layer "B.Cu") (net 20))
+  (segment (start 153.797 44.477) (end 151.7436 44.477) (width 0.25) (layer "B.Cu") (net 20))
+  (segment (start 151.7436 44.477) (end 151.511 44.2444) (width 0.25) (layer "B.Cu") (net 20))
+  (segment (start 150.725989 48.541789) (end 145.996811 48.541789) (width 0.25) (layer "B.Cu") (net 20))
+  (segment (start 150.7998 48.6156) (end 150.725989 48.541789) (width 0.25) (layer "B.Cu") (net 20))
   (segment (start 138.557 36.857) (end 134.747 36.857) (width 0.25) (layer "F.Cu") (net 21))
   (segment (start 153.797 60.5536) (end 153.797 52.097) (width 0.25) (layer "F.Cu") (net 22))
@@
   (segment (start 144.907 53.7226) (end 144.653 53.7226) (width 0.5) (layer "F.Cu") (net 23))
   (via (at 145.415 54.2814) (size 0.7) (drill 0.4) (layers "F.Cu" "B.Cu") (remove_unused_layers) (keep_end_layers) (zone_layer_connections) (net 23))
-  (segment (start 152.4 54.20928) (end 151.559694 53.368974) (width 0.75) (layer "F.Cu") (net 24))
-  (segment (start 151.559694 53.368974) (end 151.224428 53.368974) (width 0.75) (layer "F.Cu") (net 24))
-  (via (at 152.4 54.20928) (size 0.8) (drill 0.4) (layers "F.Cu" "B.Cu") (remove_unused_layers) (keep_end_layers) (free) (zone_layer_connections) (net 24))
-  (segment (start 152.4 59.595974) (end 150.914 61.081974) (width 0.75) (layer "B.Cu") (net 24))
-  (segment (start 152.4 54.20928) (end 152.4 59.595974) (width 0.75) (layer "B.Cu") (net 24))
+  (segment (start 151.363454 53.508) (end 151.224428 53.368974) (width 0.75) (layer "F.Cu") (net 24))
+  (segment (start 151.568637 53.508) (end 151.363454 53.508) (width 0.75) (layer "F.Cu") (net 24))
+  (segment (start 152.146 54.085363) (end 151.568637 53.508) (width 0.75) (layer "F.Cu") (net 24))
+  (segment (start 150.9114 61.0924) (end 152.146 59.8578) (width 0.75) (layer "F.Cu") (net 24))
+  (segment (start 152.146 59.8578) (end 152.146 54.085363) (width 0.75) (layer "F.Cu") (net 24))
   (segment (start 147.030198 54.072499) (end 147.4978 53.604897) (width 0.75) (layer "F.Cu") (net 26))
   (segment (start 147.1464 57.730077) (end 147.030198 57.613875) (width 0.75) (layer "F.Cu") (net 26))
@@
   (segment (start 148.465 55.110826) (end 148.497713 55.078113) (width 0.75) (layer "F.Cu") (net 28))
   (segment (start 148.374 58.541974) (end 148.971 57.944974) (width 0.75) (layer "F.Cu") (net 28))
+  (segment (start 151.8412 50.0888) (end 152.019 50.2666) (width 0.25) (layer "F.Cu") (net 29))
   (segment (start 152.0708 46.3312) (end 151.5354 46.8666) (width 0.25) (layer "F.Cu") (net 29))
   (segment (start 149.512988 49.524974) (end 149.3916 49.524974) (width 0.25) (layer "F.Cu") (net 29))
+  (segment (start 152.019 50.2666) (end 152.019 50.601) (width 0.25) (layer "F.Cu") (net 29))
   (segment (start 149.610303 49.622289) (end 149.512988 49.524974) (width 0.25) (layer "F.Cu") (net 29))
   (segment (start 151.5354 46.8666) (end 151.3586 46.8666) (width 0.25) (layer "F.Cu") (net 29))
@@
   (via (at 144.145 39.524) (size 0.6) (drill 0.3) (layers "F.Cu" "B.Cu") (remove_unused_layers) (keep_end_layers) (free) (zone_layer_connections "In2.Cu") (net 29))
   (via (at 143.675 54.858974) (size 0.6) (drill 0.3) (layers "F.Cu" "B.Cu") (remove_unused_layers) (keep_end_layers) (free) (zone_layer_connections "In2.Cu") (net 29))
-  (via (at 152.527 50.7762) (size 0.8) (drill 0.4) (layers "F.Cu" "B.Cu") (remove_unused_layers) (keep_end_layers) (zone_layer_connections "In2.Cu") (net 29))
+  (via (at 151.8412 50.0888) (size 0.8) (drill 0.4) (layers "F.Cu" "B.Cu") (remove_unused_layers) (keep_end_layers) (zone_layer_connections "In2.Cu") (net 29))
   (via (at 152.146 46.3312) (size 0.6) (drill 0.3) (layers "F.Cu" "B.Cu") (remove_unused_layers) (keep_end_layers) (free) (zone_layer_connections "In2.Cu") (net 29))
   (via (at 131.4958 54.383) (size 0.8) (drill 0.4) (layers "F.Cu" "B.Cu") (remove_unused_layers) (keep_end_layers) (zone_layer_connections "In2.Cu") (net 29))
@@
   (segment (start 150.05129 41.278) (end 150.497 41.72371) (width 0.25) (layer "B.Cu") (net 61))
   (segment (start 149.529892 41.278) (end 150.05129 41.278) (width 0.25) (layer "B.Cu") (net 61))
+  (zone (net 1) (net_name "GND") (layer "F.Cu") (hatch edge 0.5)
+    (priority 9)
+    (connect_pads yes (clearance 0))
+    (min_thickness 0.25) (filled_areas_thickness no)
+    (fill yes (thermal_gap 0.5) (thermal_bridge_width 0.5) (smoothing fillet) (radius 0.35))
+    (polygon
+      (pts
+        (xy 147.066 38.3032)
+        (xy 147.066 41.8592)
+        (xy 144.78 41.8592)
+        (xy 144.78 38.3032)
+      )
+    )
+  )
   (zone (net 29) (net_name "vbat") (layer "F.Cu") (hatch edge 0.5)
     (priority 11)
@@
     (connect_pads yes (clearance 0))
     (min_thickness 0.25) (filled_areas_thickness no)
-    (fill yes (thermal_gap 0.5) (thermal_bridge_width 0.5))
+    (fill yes (thermal_gap 0.5) (thermal_bridge_width 0.5) (smoothing fillet) (radius 0.35))
     (polygon
       (pts
-        (xy 144.8054 38.2778)
-        (xy 147.066 38.2778)
+        (xy 144.78 38.3032)
+        (xy 147.066 38.3032)
         (xy 147.066 41.8592)
-        (xy 144.8054 41.8592)
+        (xy 144.78 41.8592)
       )
     )

Commit message: working on v1.7
Routing:
- net GND: track 38.1 -> 39.8 mm
Other:
- board text added: "RCM Nibble v1.7"
- board text added: "v1.7"
- board text removed: "RCM Nibble v1.6"
- board text removed: "v1.6"

Commit message: v1.7
Changed lines of the file:
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@@
   (segment (start 134.747 44.477) (end 134.747 48.287) (width 0.25) (layer "F.Cu") (net 51))
   (segment (start 134.747 48.287) (end 138.557 52.097) (width 0.25) (layer "F.Cu") (net 51))
-  (segment (start 154.822 59.6318) (end 152.0638 62.39) (width 0.25) (layer "B.Cu") (net 52))
+  (segment (start 140.6656 58.6456) (end 137.8174 55.7974) (width 0.25) (layer "B.Cu") (net 52))
+  (segment (start 154.822 59.0968) (end 151.5288 62.39) (width 0.25) (layer "B.Cu") (net 52))
+  (segment (start 140.6656 61.267173) (end 140.6656 58.6456) (width 0.25) (layer "B.Cu") (net 52))
+  (segment (start 153.797 49.557) (end 154.822 50.582) (width 0.25) (layer "B.Cu") (net 52))
   (segment (start 132.9315 51.5515) (end 132.207 50.827) (width 0.25) (layer "B.Cu") (net 52))
+  (segment (start 132.9315 53.999855) (end 132.9315 51.5515) (width 0.25) (layer "B.Cu") (net 52))
+  (segment (start 141.788427 62.39) (end 140.6656 61.267173) (width 0.25) (layer "B.Cu") (net 52))
+  (segment (start 134.729045 55.7974) (end 132.9315 53.999855) (width 0.25) (layer "B.Cu") (net 52))
+  (segment (start 151.5288 62.39) (end 141.788427 62.39) (width 0.25) (layer "B.Cu") (net 52))
+  (segment (start 154.822 50.582) (end 154.822 59.0968) (width 0.25) (layer "B.Cu") (net 52))
   (segment (start 137.8174 55.7974) (end 134.729045 55.7974) (width 0.25) (layer "B.Cu") (net 52))
-  (segment (start 153.797 49.557) (end 154.822 50.582) (width 0.25) (layer "B.Cu") (net 52))
-  (segment (start 152.0638 62.39) (end 141.788427 62.39) (width 0.25) (layer "B.Cu") (net 52))
-  (segment (start 140.6656 58.6456) (end 137.8174 55.7974) (width 0.25) (layer "B.Cu") (net 52))
-  (segment (start 140.6656 61.267173) (end 140.6656 58.6456) (width 0.25) (layer "B.Cu") (net 52))
-  (segment (start 134.729045 55.7974) (end 132.9315 53.999855) (width 0.25) (layer "B.Cu") (net 52))
-  (segment (start 132.9315 53.999855) (end 132.9315 51.5515) (width 0.25) (layer "B.Cu") (net 52))
-  (segment (start 154.822 50.582) (end 154.822 59.6318) (width 0.25) (layer "B.Cu") (net 52))
-  (segment (start 141.788427 62.39) (end 140.6656 61.267173) (width 0.25) (layer "B.Cu") (net 52))
   (segment (start 145.1025 43.2185) (end 145.1025 43.7365) (width 0.2) (layer "F.Cu") (net 53))
   (segment (start 145.182 46.347) (end 145.182 45.947) (width 0.2) (layer "F.Cu") (net 53))

Commit message: v1.7.1
Parts:
- C1, C11, C15, C17, C18, C3, C4, C5, C6, C7, C8: value 100nF/0402/16V/X7R/<=10%/ceramic -> 100nF/0402/50V/X7R/<=10%/ceramic
- C16, C2, C9: value 22uF/0805/>=16V -> 22uF/0805/25V
Changed lines of the file:
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@@
         (effects (font (size 1 1) (thickness 0.15)))
     )
-    (fp_text value "22uF/0805/>=16V" (at 0 1.68) (layer "F.Fab")
+    (fp_text value "22uF/0805/25V" (at 0 1.68) (layer "F.Fab")
         (effects (font (size 1 1) (thickness 0.15)))
     )
@@
         (effects (font (size 1 1) (thickness 0.15)))
     )
-    (fp_text value "100nF/0402/16V/X7R/<=10%/ceramic" (at 0 1.16 90) (layer "F.Fab")
+    (fp_text value "100nF/0402/50V/X7R/<=10%/ceramic" (at 0 1.16 90) (layer "F.Fab")
         (effects (font (size 1 1) (thickness 0.15)))
     )
@@
         (effects (font (size 1 1) (thickness 0.15)))
     )
-    (fp_text value "100nF/0402/16V/X7R/<=10%/ceramic" (at 0 1.16) (layer "F.Fab")
+    (fp_text value "100nF/0402/50V/X7R/<=10%/ceramic" (at 0 1.16) (layer "F.Fab")
         (effects (font (size 1 1) (thickness 0.15)))
     )
@@
         (effects (font (size 1 1) (thickness 0.15)))
     )
-    (fp_text value "100nF/0402/16V/X7R/<=10%/ceramic" (at 0 1.16) (layer "F.Fab")
+    (fp_text value "100nF/0402/50V/X7R/<=10%/ceramic" (at 0 1.16) (layer "F.Fab")
         (effects (font (size 1 1) (thickness 0.15)))
     )
@@
         (effects (font (size 1 1) (thickness 0.15)))
     )
-    (fp_text value "100nF/0402/16V/X7R/<=10%/ceramic" (at 0 1.16 90) (layer "F.Fab")
+    (fp_text value "100nF/0402/50V/X7R/<=10%/ceramic" (at 0 1.16 90) (layer "F.Fab")
         (effects (font (size 1 1) (thickness 0.15)))
     )
@@
         (effects (font (size 1 1) (thickness 0.15)))
     )
-    (fp_text value "100nF/0402/16V/X7R/<=10%/ceramic" (at 0 1.16) (layer "F.Fab")
+    (fp_text value "100nF/0402/50V/X7R/<=10%/ceramic" (at 0 1.16) (layer "F.Fab")
         (effects (font (size 1 1) (thickness 0.15)))
     )
@@
         (effects (font (size 1 1) (thickness 0.15)) (justify mirror))
     )
-    (fp_text value "100nF/0402/16V/X7R/<=10%/ceramic" (at 0 -1.16 -270) (layer "B.Fab")
+    (fp_text value "100nF/0402/50V/X7R/<=10%/ceramic" (at 0 -1.16 -270) (layer "B.Fab")
         (effects (font (size 1 1) (thickness 0.15)) (justify mirror))
     )
@@
         (effects (font (size 1 1) (thickness 0.15)) (justify mirror))
     )
-    (fp_text value "22uF/0805/>=16V" (at 0 -1.68) (layer "B.Fab")
+    (fp_text value "22uF/0805/25V" (at 0 -1.68) (layer "B.Fab")
         (effects (font (size 1 1) (thickness 0.15)) (justify mirror))
     )
@@
         (effects (font (size 1 1) (thickness 0.15)) (justify mirror))
     )
-    (fp_text value "100nF/0402/16V/X7R/<=10%/ceramic" (at 0 -1.16 -270) (layer "B.Fab")
+    (fp_text value "100nF/0402/50V/X7R/<=10%/ceramic" (at 0 -1.16 -270) (layer "B.Fab")
         (effects (font (size 1 1) (thickness 0.15)) (justify mirror))
     )
@@
         (effects (font (size 1 1) (thickness 0.15)) (justify mirror))
     )
-    (fp_text value "100nF/0402/16V/X7R/<=10%/ceramic" (at 0 -1.16 90) (layer "B.Fab")
+    (fp_text value "100nF/0402/50V/X7R/<=10%/ceramic" (at 0 -1.16 90) (layer "B.Fab")
         (effects (font (size 1 1) (thickness 0.15)) (justify mirror))
     )
@@
         (effects (font (size 1 1) (thickness 0.15)) (justify mirror))
     )
-    (fp_text value "22uF/0805/>=16V" (at 0 -1.68) (layer "B.Fab")
+    (fp_text value "22uF/0805/25V" (at 0 -1.68) (layer "B.Fab")
         (effects (font (size 1 1) (thickness 0.15)) (justify mirror))
     )
@@
         (effects (font (size 1 1) (thickness 0.15)) (justify mirror))
     )
-    (fp_text value "100nF/0402/16V/X7R/<=10%/ceramic" (at 0 -1.16 90) (layer "B.Fab")
+    (fp_text value "100nF/0402/50V/X7R/<=10%/ceramic" (at 0 -1.16 90) (layer "B.Fab")
         (effects (font (size 1 1) (thickness 0.15)) (justify mirror))
     )
@@
         (effects (font (size 1 1) (thickness 0.15)) (justify mirror))
     )
-    (fp_text value "100nF/0402/16V/X7R/<=10%/ceramic" (at 0 -1.16 90) (layer "B.Fab")
+    (fp_text value "100nF/0402/50V/X7R/<=10%/ceramic" (at 0 -1.16 90) (layer "B.Fab")
         (effects (font (size 1 1) (thickness 0.15)) (justify mirror))
     )
@@
         (effects (font (size 1 1) (thickness 0.15)) (justify mirror))
     )
-    (fp_text value "100nF/0402/16V/X7R/<=10%/ceramic" (at 0 -1.16) (layer "B.Fab")
-        (effects (font (size 1 1) (thickness 0.15)) (justify mirror))
-    )
+    (fp_text value "100nF/0402/50V/X7R/<=10%/ceramic" (at 0 -1.16) (layer "B.Fab")
+        (effects (font (size 1 1) (thickness 0.15)) (justify mirror))
+    )

Commit message: v1.8
Parts:
- moved U2 1.01 mm to (145.9, 41.0), turned to 180 degrees
- moved U1 0.05 mm to (140.0, 34.4)
Routing:
- net Net-(Q3-S): track 6.18 -> 5.44 mm
- net Net-(IC2-1,8Vout): track 1.17 -> 1.88 mm
