File: KICAD-RCM-Nibble/RCMhardwareNibble.kicad_pcb (KiCad board)
At the start: 4 copper layers, 27.4 x 28.4 mm, 51 parts, among them IC1 TMC7300, IC2 TMC7300, J1 pads to solder wires to, J2 Conn_01x03, J3 Conn_01x03, J4 Conn_01x03, J5 Conn_01x03, J6 2x04 female header pins, J9 Conn_02x02_Top_Bottom, Q3 BSS138, N channel mosfet >=0.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

Commit message: v1.8
Other:
- board text added: "RCM Nibble v1.8"
- board text added: "v1.8"
- board text removed: "RCM Nibble v1.7"
- board text removed: "v1.7"
Changed lines of the file:
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@@
     (effects (font (size 2 2) (thickness 0.3)) (justify mirror))
   )
-  (gr_text "RCM Nibble v1.7\n" (at 150.6982 49.0474) (layer "B.SilkS")
+  (gr_text "RCM Nibble v1.8\n" (at 150.6982 49.0474) (layer "B.SilkS")
     (effects (font (size 0.8 0.8) (thickness 0.15)) (justify left bottom mirror))
   )
@@
     (effects (font (size 0.9 0.9) (thickness 0.15)) (justify left bottom))
   )
-  (gr_text "v1.7\n" (at 134.5946 50.1666) (layer "F.SilkS")
+  (gr_text "v1.8\n" (at 134.5946 50.1666) (layer "F.SilkS")
     (effects (font (size 0.8 0.8) (thickness 0.15)) (justify left bottom))
   )
