File: KICAD-RCM-Nibble/RCMhardwareNibble.kicad_sch (KiCad schematic)
At the start: 51 parts, among them IC1 TMC7300, IC2 TMC7300, J1 pads to solder wires to, J2 Conn_01x03, J3 Conn_01x03, J4 Conn_01x03, J5 Conn_01x03, J6 2x04 female header pins, J9 Conn_02x02_Top_Bottom, Q3 BSS138, N channel mosfet >=0.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

Commit message: v1.7
Parts:
- H1, H2: mpn n/a -> DNP
- Q3, Q4: Manufacturer any -> onsemi
- R1, R10, R11, R12, R13, R2, R3, R4, R5, R6, R7, R9: Manufacturer any -> Bourns Inc.
Changed lines of the file:
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@@
   (title_block
     (title "RCM NIBBLE")
-    (rev "1.6")
+    (rev "1.7")
     (company "RCMgames")
     (comment 1 "https://github.com/RCMgames/RCM-Hardware-Nibble")
@@
       (effects (font (size 1.27 1.27)) hide)
     )
-    (property "Manufacturer" "any" (at 143.51 180.34 0)
+    (property "Manufacturer" "Bourns Inc." (at 143.51 180.34 0)
       (effects (font (size 1.27 1.27)) hide)
     )
@@
       (effects (font (size 1.27 1.27)) hide)
     )
-    (property "Manufacturer" "any" (at 303.53 163.83 0)
+    (property "Manufacturer" "Bourns Inc." (at 303.53 163.83 0)
       (effects (font (size 1.27 1.27)) hide)
     )
@@
       (effects (font (size 1.27 1.27)) hide)
     )
-    (property "Manufacturer" "any" (at 288.29 181.61 0)
+    (property "Manufacturer" "onsemi" (at 288.29 181.61 0)
       (effects (font (size 1.27 1.27)) hide)
     )
@@
       (effects (font (size 1.27 1.27) italic) hide)
     )
-    (property "Datasheet" "LTC3246EMSE-PBF" (at 372.11 290.83 0)
+    (property "Datasheet" "~" (at 372.11 290.83 0)
       (effects (font (size 1.27 1.27) italic) hide)
     )
@@
       (effects (font (size 1.27 1.27)) hide)
     )
-    (property "Manufacturer" "any" (at 439.42 295.91 0)
+    (property "Manufacturer" "Bourns Inc." (at 439.42 295.91 0)
       (effects (font (size 1.27 1.27)) hide)
     )
@@
       (effects (font (size 1.27 1.27)) hide)
     )
-    (property "Manufacturer" "any" (at 142.24 88.9 0)
+    (property "Manufacturer" "Bourns Inc." (at 142.24 88.9 0)
       (effects (font (size 1.27 1.27)) hide)
     )
@@
       (effects (font (size 1.27 1.27)) hide)
     )
-    (property "mpn" "n/a" (at 466.09 134.62 0)
+    (property "mpn" "DNP" (at 466.09 134.62 0)
       (effects (font (size 1.27 1.27)) hide)
     )
@@
       (effects (font (size 1.27 1.27)) hide)
     )
-    (property "Manufacturer" "any" (at 379.73 40.64 0)
+    (property "Manufacturer" "Bourns Inc." (at 379.73 40.64 0)
       (effects (font (size 1.27 1.27)) hide)
     )
@@
       (effects (font (size 1.27 1.27)) hide)
     )
-    (property "mpn" "n/a" (at 466.09 128.27 0)
+    (property "mpn" "DNP" (at 466.09 128.27 0)
       (effects (font (size 1.27 1.27)) hide)
     )
@@
       (effects (font (size 1.27 1.27)) hide)
     )
-    (property "Manufacturer" "any" (at 276.86 162.56 0)
+    (property "Manufacturer" "Bourns Inc." (at 276.86 162.56 0)
       (effects (font (size 1.27 1.27)) hide)
     )
@@
       (effects (font (size 1.27 1.27)) hide)
     )
-    (property "Manufacturer" "any" (at 143.51 162.56 0)
+    (property "Manufacturer" "Bourns Inc." (at 143.51 162.56 0)
       (effects (font (size 1.27 1.27)) hide)
     )
@@
       (effects (font (size 1.27 1.27)) hide)
     )
-    (property "Manufacturer" "any" (at 389.89 39.37 0)
+    (property "Manufacturer" "Bourns Inc." (at 389.89 39.37 0)
       (effects (font (size 1.27 1.27)) hide)
     )
@@
       (effects (font (size 1.27 1.27)) hide)
     )
-    (property "Manufacturer" "any" (at 303.53 190.5 0)
+    (property "Manufacturer" "Bourns Inc." (at 303.53 190.5 0)
       (effects (font (size 1.27 1.27)) hide)
     )
@@
       (effects (font (size 1.27 1.27)) hide)
     )
-    (property "Manufacturer" "any" (at 433.07 85.09 0)
+    (property "Manufacturer" "Bourns Inc." (at 433.07 85.09 0)
       (effects (font (size 1.27 1.27)) hide)
     )
@@
       (effects (font (size 1.27 1.27)) hide)
     )
-    (property "Manufacturer" "any" (at 288.29 165.1 0)
+    (property "Manufacturer" "onsemi" (at 288.29 165.1 0)
       (effects (font (size 1.27 1.27)) hide)
     )
@@
       (effects (font (size 1.27 1.27)) hide)
     )
-    (property "Manufacturer" "any" (at 276.86 182.88 0)
+    (property "Manufacturer" "Bourns Inc." (at 276.86 182.88 0)
       (effects (font (size 1.27 1.27)) hide)
     )
@@
       (effects (font (size 1.27 1.27)) hide)
     )
-    (property "Manufacturer" "any" (at 142.24 71.12 0)
+    (property "Manufacturer" "Bourns Inc." (at 142.24 71.12 0)
       (effects (font (size 1.27 1.27)) hide)
     )

Commit message: v1.7.0
Parts:
- C1, C10, C11, C12, C13, C14, C15, C16, C17, C18, C2, C3, C4, C5, C6, C7, C8, C9: Manufacturer any -> Cal-Chip Electronics, Inc.
Changed lines of the file:
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@@
       (effects (font (size 1.27 1.27)) hide)
     )
-    (property "Manufacturer" "any" (at 387.35 142.24 0)
+    (property "Manufacturer" "Cal-Chip Electronics, Inc." (at 387.35 142.24 0)
       (effects (font (size 1.27 1.27)) hide)
     )
@@
       (effects (font (size 1.27 1.27)) hide)
     )
-    (property "Manufacturer" "any" (at 440.69 302.26 0)
+    (property "Manufacturer" "Cal-Chip Electronics, Inc." (at 440.69 302.26 0)
       (effects (font (size 1.27 1.27)) hide)
     )
@@
       (effects (font (size 1.27 1.27)) hide)
     )
-    (property "Manufacturer" "any" (at 90.17 109.22 0)
+    (property "Manufacturer" "Cal-Chip Electronics, Inc." (at 90.17 109.22 0)
       (effects (font (size 1.27 1.27)) hide)
     )
@@
       (effects (font (size 1.27 1.27)) hide)
     )
-    (property "Manufacturer" "any" (at 69.85 72.39 0)
+    (property "Manufacturer" "Cal-Chip Electronics, Inc." (at 69.85 72.39 0)
       (effects (font (size 1.27 1.27)) hide)
     )
@@
       (effects (font (size 1.27 1.27)) hide)
     )
-    (property "Manufacturer" "any" (at 97.79 157.48 0)
+    (property "Manufacturer" "Cal-Chip Electronics, Inc." (at 97.79 157.48 0)
       (effects (font (size 1.27 1.27)) hide)
     )
@@
       (effects (font (size 1.27 1.27)) hide)
     )
-    (property "Manufacturer" "any" (at 372.11 312.42 0)
+    (property "Manufacturer" "Cal-Chip Electronics, Inc." (at 372.11 312.42 0)
       (effects (font (size 1.27 1.27)) hide)
     )
@@
       (effects (font (size 1.27 1.27)) hide)
     )
-    (property "Manufacturer" "any" (at 137.16 111.76 0)
+    (property "Manufacturer" "Cal-Chip Electronics, Inc." (at 137.16 111.76 0)
       (effects (font (size 1.27 1.27)) hide)
     )
@@
       (effects (font (size 1.27 1.27)) hide)
     )
-    (property "Manufacturer" "any" (at 95.25 66.04 0)
+    (property "Manufacturer" "Cal-Chip Electronics, Inc." (at 95.25 66.04 0)
       (effects (font (size 1.27 1.27)) hide)
     )
@@
       (effects (font (size 1.27 1.27)) hide)
     )
-    (property "Manufacturer" "any" (at 351.79 171.45 0)
+    (property "Manufacturer" "Cal-Chip Electronics, Inc." (at 351.79 171.45 0)
       (effects (font (size 1.27 1.27)) hide)
     )
@@
       (effects (font (size 1.27 1.27)) hide)
     )
-    (property "Manufacturer" "any" (at 429.26 64.77 0)
+    (property "Manufacturer" "Cal-Chip Electronics, Inc." (at 429.26 64.77 0)
       (effects (font (size 1.27 1.27)) hide)
     )
@@
       (effects (font (size 1.27 1.27)) hide)
     )
-    (property "Manufacturer" "any" (at 71.12 163.83 0)
+    (property "Manufacturer" "Cal-Chip Electronics, Inc." (at 71.12 163.83 0)
       (effects (font (size 1.27 1.27)) hide)
     )
@@
       (effects (font (size 1.27 1.27)) hide)
     )
-    (property "Manufacturer" "any" (at 454.66 308.61 0)
+    (property "Manufacturer" "Cal-Chip Electronics, Inc." (at 454.66 308.61 0)
       (effects (font (size 1.27 1.27)) hide)
     )
@@
       (effects (font (size 1.27 1.27)) hide)
     )
-    (property "Manufacturer" "any" (at 91.44 200.66 0)
+    (property "Manufacturer" "Cal-Chip Electronics, Inc." (at 91.44 200.66 0)
       (effects (font (size 1.27 1.27)) hide)
     )
@@
       (effects (font (size 1.27 1.27)) hide)
     )
-    (property "Manufacturer" "any" (at 280.67 82.55 0)
+    (property "Manufacturer" "Cal-Chip Electronics, Inc." (at 280.67 82.55 0)
       (effects (font (size 1.27 1.27)) hide)
     )
@@
       (effects (font (size 1.27 1.27)) hide)
     )
-    (property "Manufacturer" "any" (at 427.99 314.96 0)
+    (property "Manufacturer" "Cal-Chip Electronics, Inc." (at 427.99 314.96 0)
       (effects (font (size 1.27 1.27)) hide)
     )
@@
       (effects (font (size 1.27 1.27)) hide)
     )
-    (property "Manufacturer" "any" (at 436.88 58.42 0)
+    (property "Manufacturer" "Cal-Chip Electronics, Inc." (at 436.88 58.42 0)
       (effects (font (size 1.27 1.27)) hide)
     )
@@
       (effects (font (size 1.27 1.27)) hide)
     )
-    (property "Manufacturer" "any" (at 421.64 54.61 0)
+    (property "Manufacturer" "Cal-Chip Electronics, Inc." (at 421.64 54.61 0)
       (effects (font (size 1.27 1.27)) hide)
     )
@@
       (effects (font (size 1.27 1.27)) hide)
     )
-    (property "Manufacturer" "any" (at 138.43 203.2 0)
-      (effects (font (size 1.27 1.27)) hide)
-    )
+    (property "Manufacturer" "Cal-Chip Electronics, Inc." (at 138.43 203.2 0)
+      (effects (font (size 1.27 1.27)) hide)
+    )

Commit message: v1.7.1
Parts:
- C1, C11, C15, C17, C18, C3, C4, C5, C6, C7, C8: value 100nF/0402/16V/X7R/<=10%/ceramic -> 100nF/0402/50V/X7R/<=10%/ceramic
- C16, C2, C9: value 22uF/0805/>=16V -> 22uF/0805/25V
Changed lines of the file:
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@@
       (effects (font (size 0.9906 0.9906)))
     )
-    (property "Value" "100nF/0402/16V/X7R/<=10%/ceramic" (at 93.98 109.22 90)
+    (property "Value" "100nF/0402/50V/X7R/<=10%/ceramic" (at 93.98 109.22 90)
       (effects (font (size 0.9906 0.9906)))
     )
@@
       (effects (font (size 0.9906 0.9906)))
     )
-    (property "Value" "100nF/0402/16V/X7R/<=10%/ceramic" (at 73.66 72.39 90)
+    (property "Value" "100nF/0402/50V/X7R/<=10%/ceramic" (at 73.66 72.39 90)
       (effects (font (size 0.9906 0.9906)))
     )
@@
       (effects (font (size 0.9906 0.9906)))
     )
-    (property "Value" "100nF/0402/16V/X7R/<=10%/ceramic" (at 96.52 149.86 90)
+    (property "Value" "100nF/0402/50V/X7R/<=10%/ceramic" (at 96.52 149.86 90)
       (effects (font (size 0.9906 0.9906)))
     )
@@
       (effects (font (size 1.27 1.27)) (justify right))
     )
-    (property "Value" "22uF/0805/>=16V" (at 374.65 313.69 0)
+    (property "Value" "22uF/0805/25V" (at 374.65 313.69 0)
       (effects (font (size 1.27 1.27)) (justify right))
     )
@@
       (effects (font (size 0.9906 0.9906)))
     )
-    (property "Value" "100nF/0402/16V/X7R/<=10%/ceramic" (at 140.97 111.76 90)
+    (property "Value" "100nF/0402/50V/X7R/<=10%/ceramic" (at 140.97 111.76 90)
       (effects (font (size 0.9906 0.9906)))
     )
@@
       (effects (font (size 0.9906 0.9906)))
     )
-    (property "Value" "100nF/0402/16V/X7R/<=10%/ceramic" (at 93.98 60.96 90)
+    (property "Value" "100nF/0402/50V/X7R/<=10%/ceramic" (at 93.98 60.96 90)
       (effects (font (size 0.9906 0.9906)))
     )
@@
       (effects (font (size 0.9906 0.9906)))
     )
-    (property "Value" "100nF/0402/16V/X7R/<=10%/ceramic" (at 369.57 171.45 0)
+    (property "Value" "100nF/0402/50V/X7R/<=10%/ceramic" (at 369.57 171.45 0)
       (effects (font (size 0.9906 0.9906)))
     )
@@
       (effects (font (size 1.27 1.27)) (justify left))
     )
-    (property "Value" "22uF/0805/>=16V" (at 433.07 66.04 0)
+    (property "Value" "22uF/0805/25V" (at 433.07 66.04 0)
       (effects (font (size 1.27 1.27)) (justify left))
     )
@@
       (effects (font (size 0.9906 0.9906)))
     )
-    (property "Value" "100nF/0402/16V/X7R/<=10%/ceramic" (at 74.93 163.83 90)
+    (property "Value" "100nF/0402/50V/X7R/<=10%/ceramic" (at 74.93 163.83 90)
       (effects (font (size 0.9906 0.9906)))
     )
@@
       (effects (font (size 0.9906 0.9906)))
     )
-    (property "Value" "100nF/0402/16V/X7R/<=10%/ceramic" (at 95.25 201.93 90)
+    (property "Value" "100nF/0402/50V/X7R/<=10%/ceramic" (at 95.25 201.93 90)
       (effects (font (size 0.9906 0.9906)))
     )
@@
       (effects (font (size 0.9906 0.9906)))
     )
-    (property "Value" "100nF/0402/16V/X7R/<=10%/ceramic" (at 275.59 82.55 90)
+    (property "Value" "100nF/0402/50V/X7R/<=10%/ceramic" (at 275.59 82.55 90)
       (effects (font (size 0.9906 0.9906)))
     )
@@
       (effects (font (size 1.27 1.27)) (justify left))
     )
-    (property "Value" "22uF/0805/>=16V" (at 440.69 59.69 0)
+    (property "Value" "22uF/0805/25V" (at 440.69 59.69 0)
       (effects (font (size 1.27 1.27)) (justify left))
     )
@@
       (effects (font (size 0.9906 0.9906)))
     )
-    (property "Value" "100nF/0402/16V/X7R/<=10%/ceramic" (at 424.18 60.96 90)
+    (property "Value" "100nF/0402/50V/X7R/<=10%/ceramic" (at 424.18 60.96 90)
       (effects (font (size 0.9906 0.9906)))
     )
@@
       (effects (font (size 0.9906 0.9906)))
     )
-    (property "Value" "100nF/0402/16V/X7R/<=10%/ceramic" (at 142.24 203.2 90)
-      (effects (font (size 0.9906 0.9906)))
-    )
+    (property "Value" "100nF/0402/50V/X7R/<=10%/ceramic" (at 142.24 203.2 90)
+      (effects (font (size 0.9906 0.9906)))
+    )

Commit message: update production files
Parts:
- U3: mount_type smt -> smt (do not solder center pad)
Changed lines of the file:
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@@
       (effects (font (size 1.27 1.27)) hide)
     )
-    (property "mount_type" "smt" (at 326.39 171.45 0)
+    (property "mount_type" "smt (do not solder center pad)" (at 326.39 171.45 0)
       (effects (font (size 1.27 1.27)) hide)
     )
